Commit message: gen3 ik solving 오류 개선

File: ros2_ws/src/ros2_kortex/kortex_description/robots/gen3_7dof.urdf (robot description, URDF)
Before this commit: robot gen3-7dof, 9 links, 8 joints
Joints:
- joint joint_1: limit effort=39 velocity=1.3963 -> lower=-3.14159 upper=3.14159 effort=39 velocity=1.3963
- joint joint_3: limit effort=39 velocity=1.3963 -> lower=-3.14159 upper=3.14159 effort=39 velocity=1.3963
- joint joint_5: limit effort=9 velocity=1.2218 -> lower=-3.14159 upper=3.14159 effort=39 velocity=1.3963
- joint joint_7: limit effort=9 velocity=1.2218 -> lower=-3.14159 upper=3.14159 effort=39 velocity=1.3963
